Commit message: Fix camera pitch

File: bot_description/urdf/bot_front_wheels.urdf (robot description, URDF)
Before this commit: robot bot, 7 links, 6 joints
Joints:
- joint axletocameraplate: origin xyz=0.05308 0 0.03633 rpy=0 -0.297 0 -> xyz=0.05308 0 0.03633 rpy=0 -0.349 0
- joint cameratolaser: origin xyz=0 0 0 rpy=0 0.297 0 -> xyz=0 0 0 rpy=0 0.349 0

Commit message: Switch to lidar

File: bot_description/urdf/bot_front_wheels.urdf (robot description, URDF)
Before this commit: robot bot, 7 links, 6 joints
Joints:
- joint axletocameraplate: origin xyz=0.05308 0 0.03633 rpy=0 -0.349 0 -> xyz=0.05308 0 0.03633 rpy=0 0 0
- joint camerainternaloffset: origin xyz=-0.00420 0.01750 0 rpy=0 0 0 -> xyz=-0.00420 0.01750 0 rpy=0 0 3.14156
- joint cameratolaser: origin xyz=0 0 0 rpy=0 0.349 0 -> xyz=0 0 0 rpy=0 0 0
